File: Hardware/Host/pico_pmod_host.kicad_pcb (KiCad board)
At the start: 2 copper layers, 66 x 43.2 mm, 8 parts, among them J1 Conn_02x15_Odd_Even, J2 Conn_01x02, J3 Conn_01x02, J4 Conn_01x02, J5 Conn_01x03, J7 Conn_01x05, SW1 SW_Push, U1 Pico

Commit message: update the 5v pinout on the pmod connector for #1 on the PCB
Connections:
- J1 pad 15: GND -> +5V
- J1 pad 16: +5V -> GND
Routing:
- net GND: track 1.28 -> 14.6 mm, vias 3 -> 4
- net +5V: track 81.4 -> 72.5 mm
- net GPIO_16: track 17.1 -> 17.9 mm, vias 0 -> 1

Commit message: Change the logo on the host board
Parts:
- added G***: LOGO, jjh:ContactDetails_small, B.Cu at (147.3, 85.7)
- added G***: LOGO, jjh:Untitled, B.Cu at (152.6, 102.7)
Other:
- board text added: "Raspberry Pi Pico PMod Host"
- board text removed: "Raspberry Pi Pico PMod Host @JamesjHorton JJHorton.co.uk"
