File: Hardware/Custom/pico_pmod.sch (KiCad schematic (older format))
At the start: 39 parts, among them J1 Conn_02x06_Odd_Even, J2 Conn_02x06_Odd_Even, J3 Conn_02x06_Odd_Even, J4 USB_C_Receptacle_USB2.0, J5 Conn_01x04, SW1 SW_Push, SW2 SW_Push, U1 RP2040, U2 W25Q128JVS, U3 NCP1117-3.3_SOT223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

Commit message: Correct USB DP and DN for #7
Connections:
- net USB_DP: now also R3.1; no longer R4.1
- net USB_DN renamed USB_DM
- net USB_DM: now also R4.1; no longer R3.1
Changed lines of the file:
@@
 USB_DP
 Text GLabel 2400 6450 2    51   Input ~ 0
-USB_DN
+USB_DM
 Wire Wire Line
 	1900 6450 2150 6450
@@
 	7100 1750 7250 1750
 Text GLabel 7700 1900 2    51   Input ~ 0
+USB_DM
+Text GLabel 7700 1750 2    51   Input ~ 0
 USB_DP
-Text GLabel 7700 1750 2    51   Input ~ 0
-USB_DN
 Wire Wire Line
 	7700 1750 7550 1750
