File: Hardware/RP2040_PMod/pico_pmod.sch (KiCad schematic (older format))
At the start: 39 parts, among them J1 Conn_02x06_Odd_Even, J2 Conn_02x06_Odd_Even, J3 Conn_02x06_Odd_Even, J4 USB_C_Receptacle_USB2.0, J5 Conn_01x04, SW1 SW_Push, SW2 SW_Push, U1 RP2040, U2 W25Q128JVS, U3 NCP1117-3.3_SOT223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

Commit message: Update the clk Caps
Parts:
- C2, C4: value 20p -> 10p
Changed lines of the file:
@@
 P 1300 3250
 F 0 "C2" H 1000 3300 50  0000 L CNN
-F 1 "20p" H 1000 3200 50  0000 L CNN
+F 1 "10p" H 1000 3200 50  0000 L CNN
 F 2 "Capacitor_SMD:C_0603_1608Metric" H 1338 3100 50  0001 C CNN
 F 3 "~" H 1300 3250 50  0001 C CNN
@@
 P 2100 3250
 F 0 "C4" H 2215 3296 50  0000 L CNN
-F 1 "20p" H 2215 3205 50  0000 L CNN
+F 1 "10p" H 2215 3205 50  0000 L CNN
 F 2 "Capacitor_SMD:C_0603_1608Metric" H 2138 3100 50  0001 C CNN
 F 3 "~" H 2100 3250 50  0001 C CNN
