File: Hardware/RP2040_PMod/pico_pmod.kicad_pcb (KiCad board)
At the start: 2 copper layers, 50 x 37 mm, 45 parts, among them J1 Conn_02x06_Odd_Even, J2 Conn_02x06_Odd_Even, J3 Conn_02x06_Odd_Even, J4 USB_C_Receptacle_USB2.0, J5 Conn_01x04, SW1 SW_Push, SW2 SW_Push, U1 RP2040, U2 W25Q128JVS, U3 NCP1117-3.3_SOT223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

Commit message: remove the Ref on the holes
Parts:
- renumbered REF** to Hole1, REF** to Hole2, REF** to Hole3, REF** to Hole4
Changed lines of the file:
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@@
     (tags "mounting hole 2.2mm no annular m2")
     (attr exclude_from_pos_files exclude_from_bom)
-    (fp_text reference "REF**" (at 0 -3.2) (layer "F.SilkS") hide
+    (fp_text reference "Hole1" (at 0 -3.2) (layer "F.SilkS") hide
         (effects (font (size 1 1) (thickness 0.15)))
     )
@@
     (tags "mounting hole 2.2mm no annular m2")
     (attr exclude_from_pos_files exclude_from_bom)
-    (fp_text reference "REF**" (at 0 -3.2) (layer "F.SilkS") hide
+    (fp_text reference "Hole3" (at 0 -3.2) (layer "F.SilkS") hide
         (effects (font (size 1 1) (thickness 0.15)))
     )
@@
     (tags "mounting hole 2.2mm no annular m2")
     (attr exclude_from_pos_files exclude_from_bom)
-    (fp_text reference "REF**" (at 0 -3.2) (layer "F.SilkS") hide
+    (fp_text reference "Hole2" (at 0 -3.2) (layer "F.SilkS") hide
         (effects (font (size 1 1) (thickness 0.15)))
     )
@@
     (tags "mounting hole 2.2mm no annular m2")
     (attr exclude_from_pos_files exclude_from_bom)
-    (fp_text reference "REF**" (at 0 -3.2) (layer "F.SilkS") hide
+    (fp_text reference "Hole4" (at 0 -3.2) (layer "F.SilkS") hide
         (effects (font (size 1 1) (thickness 0.15)))
     )

Commit message: change logo designator
Parts:
- renumbered G*** to L1, G*** to L2
Changed lines of the file:
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@@
     (at 157 81.25)
     (attr through_hole)
-    (fp_text reference "G***" (at 0 0) (layer "F.SilkS") hide
+    (fp_text reference "L1" (at 0 0) (layer "F.SilkS") hide
         (effects (font (size 1.524 1.524) (thickness 0.3)))
     )
@@
     (at 154.5 74.7 180)
     (attr through_hole)
-    (fp_text reference "G***" (at 0 0) (layer "F.SilkS") hide
+    (fp_text reference "L2" (at 0 0) (layer "F.SilkS") hide
         (effects (font (size 1.524 1.524) (thickness 0.3)))
     )
