File: Hardware/RP2040_PMod/pico_pmod.kicad_sch (KiCad schematic)
At the start: 39 parts, among them J1 Conn_02x06_Odd_Even, J2 Conn_02x06_Odd_Even, J3 Conn_02x06_Odd_Even, J4 USB_C_Receptacle_USB2.0, J5 Conn_01x04, SW1 SW_Push, SW2 SW_Push, U1 RP2040, U2 W25Q128JVS, U3 NCP1117-3.3_SOT223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

Commit message: update to include more components
Parts:
- C1: JLC C23630 -> (none); LCSC# (none) -> C23630
- C10, C11, C12, C3, C5, C6, C7, C8, C9: JLC C14663 -> (none); LCSC# (none) -> C14663
- C13, C14: JLC C19702 -> (none); LCSC# (none) -> C19702
- C15, C16: JLC C15849 -> (none); LCSC# (none) -> C15849
- C2, C4: JLC C1634 -> (none); LCSC# (none) -> C1634
- D1, D2, D3: JLC C2286 -> (none); LCSC# (none) -> C2286
- J4: JLC C5119948 -> (none); LCSC# (none) -> C5119948
- R2: JLC C21190 -> (none); LCSC# (none) -> C21190
- R5, R6: JLC C23186 -> (none); LCSC# (none) -> C23186
- R7, R8, R9: JLC C23138 -> (none); LCSC# (none) -> C23138
- U2: JLC C97521 -> (none); LCSC# (none) -> C97521
- U3: JLC C146799 -> (none); LCSC# (none) -> C146799
- Y1: JLC C5765982 -> (none); LCSC# (none) -> C5765982
Changed lines of the file:
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@@
       (effects (font (size 1.27 1.27)) hide)
     )
-    (property "JLC" "C21190" (at 97.79 175.26 0)
+    (property "LCSC#" "C21190" (at 97.79 175.26 0)
       (effects (font (size 1.27 1.27)) hide)
     )
@@
       (effects (font (size 1.27 1.27)) hide)
     )
-    (property "JLC" "C5119948" (at 33.02 166.37 0)
+    (property "LCSC#" "C5119948" (at 33.02 166.37 0)
       (effects (font (size 1.27 1.27)) hide)
     )
@@
       (effects (font (size 1.27 1.27)) hide)
     )
-    (property "JLC" "C97521" (at 43.18 124.46 0)
+    (property "LCSC#" "C97521" (at 43.18 124.46 0)
       (effects (font (size 1.27 1.27)) hide)
     )
@@
       (effects (font (size 1.27 1.27)) hide)
     )
-    (property "JLC" "C5765982" (at 43.18 78.74 0)
+    (property "LCSC#" "C5765982" (at 43.18 78.74 0)
       (effects (font (size 1.27 1.27)) hide)
     )
@@
       (effects (font (size 1.27 1.27)) hide)
     )
-    (property "JLC" "C146799" (at 248.92 147.32 0)
+    (property "LCSC#" "C146799" (at 248.92 147.32 0)
       (effects (font (size 1.27 1.27)) hide)
     )
@@
       (effects (font (size 1.27 1.27)) hide)
     )
-    (property "JLC" "C14663" (at 26.67 107.95 0)
+    (property "LCSC#" "C14663" (at 26.67 107.95 0)
       (effects (font (size 1.27 1.27)) hide)
     )
@@
       (effects (font (size 1.27 1.27)) hide)
     )
-    (property "JLC" "C23630" (at 16.51 107.95 0)
+    (property "LCSC#" "C23630" (at 16.51 107.95 0)
       (effects (font (size 1.27 1.27)) hide)
     )
@@
       (effects (font (size 1.27 1.27)) hide)
     )
-    (property "JLC" "C19702" (at 275.59 151.13 0)
+    (property "LCSC#" "C19702" (at 275.59 151.13 0)
       (effects (font (size 1.27 1.27)) hide)
     )
@@
       (effects (font (size 1.27 1.27)) hide)
     )
-    (property "JLC" "C19702" (at 218.44 151.13 0)
+    (property "LCSC#" "C19702" (at 218.44 151.13 0)
       (effects (font (size 1.27 1.27)) hide)
     )
@@
       (effects (font (size 1.27 1.27)) hide)
     )
-    (property "JLC" "C15849" (at 93.98 26.67 0)
+    (property "LCSC#" "C15849" (at 93.98 26.67 0)
       (effects (font (size 1.27 1.27)) hide)
     )
@@
       (effects (font (size 1.27 1.27)) hide)
     )
+    (property "LCSC#" "" (at 187.96 44.45 90)
+      (effects (font (size 1.27 1.27)) hide)
+    )
     (pin "1")
     (pin "2")
@@
       (effects (font (size 1.27 1.27)) hide)
     )
+    (property "LCSC#" "" (at 187.96 48.26 90)
+      (effects (font (size 1.27 1.27)) hide)
+    )
     (pin "1")
     (pin "2")
@@
       (effects (font (size 1.27 1.27)) hide)
     )
-    (property "JLC" "C23186" (at 57.15 156.21 90)
+    (property "LCSC#" "C23186" (at 57.15 156.21 90)
       (effects (font (size 1.27 1.27)) hide)
     )
@@
       (effects (font (size 1.27 1.27)) hide)
     )
-    (property "JLC" "C23186" (at 57.15 158.75 90)
+    (property "LCSC#" "C23186" (at 57.15 158.75 90)
       (effects (font (size 1.27 1.27)) hide)
     )
@@
       (effects (font (size 1.27 1.27)) hide)
     )
-    (property "JLC" "C15849" (at 198.12 20.32 0)
+    (property "LCSC#" "C15849" (at 198.12 20.32 0)
       (effects (font (size 1.27 1.27)) hide)
     )
@@
       (effects (font (size 1.27 1.27)) hide)
     )
-    (property "JLC" "C1634" (at 33.02 82.55 0)
+    (property "LCSC#" "C1634" (at 33.02 82.55 0)
       (effects (font (size 1.27 1.27)) hide)
     )
@@
       (effects (font (size 1.27 1.27)) hide)
     )
-    (property "JLC" "C1634" (at 53.34 82.55 0)
+    (property "LCSC#" "C1634" (at 53.34 82.55 0)
       (effects (font (size 1.27 1.27)) hide)
     )
@@
       (effects (font (size 1.27 1.27)) hide)
     )
-    (property "JLC" "C23138" (at 227.33 110.49 0)
+    (property "LCSC#" "C23138" (at 227.33 110.49 0)
       (effects (font (size 1.27 1.27)) hide)
     )
@@
       (effects (font (size 1.27 1.27)) hide)
     )
-    (property "JLC" "C2286" (at 227.33 118.11 90)
+    (property "LCSC#" "C2286" (at 227.33 118.11 90)
       (effects (font (size 1.27 1.27)) hide)
     )
@@
       (effects (font (size 1.27 1.27)) hide)
     )
-    (property "JLC" "C23138" (at 247.65 110.49 0)
+    (property "LCSC#" "C23138" (at 247.65 110.49 0)
       (effects (font (size 1.27 1.27)) hide)
     )
@@
       (effects (font (size 1.27 1.27)) hide)
     )
-    (property "JLC" "C2286" (at 247.65 118.11 90)
+    (property "LCSC#" "C2286" (at 247.65 118.11 90)
       (effects (font (size 1.27 1.27)) hide)
     )
@@
       (effects (font (size 1.27 1.27)) hide)
     )
-    (property "JLC" "C23138" (at 273.05 109.22 0)
+    (property "LCSC#" "C23138" (at 273.05 109.22 0)
       (effects (font (size 1.27 1.27)) hide)
     )
@@
       (effects (font (size 1.27 1.27)) hide)
     )
-    (property "JLC" "C2286" (at 273.05 116.84 90)
+    (property "LCSC#" "C2286" (at 273.05 116.84 90)
       (effects (font (size 1.27 1.27)) hide)
     )
@@
       (effects (font (size 1.27 1.27)) hide)
     )
-    (property "JLC" "C14663" (at 102.87 26.67 0)
+    (property "LCSC#" "C14663" (at 102.87 26.67 0)
       (effects (font (size 1.27 1.27)) hide)
     )
@@
       (effects (font (size 1.27 1.27)) hide)
     )
-    (property "JLC" "C14663" (at 111.76 26.67 0)
+    (property "LCSC#" "C14663" (at 111.76 26.67 0)
       (effects (font (size 1.27 1.27)) hide)
     )
@@
       (effects (font (size 1.27 1.27)) hide)
     )
-    (property "JLC" "C14663" (at 147.32 20.32 0)
+    (property "LCSC#" "C14663" (at 147.32 20.32 0)
       (effects (font (size 1.27 1.27)) hide)
     )
@@
       (effects (font (size 1.27 1.27)) hide)
     )
-    (property "JLC" "C14663" (at 156.21 20.32 0)
+    (property "LCSC#" "C14663" (at 156.21 20.32 0)
       (effects (font (size 1.27 1.27)) hide)
     )
@@
       (effects (font (size 1.27 1.27)) hide)
     )
-    (property "JLC" "C14663" (at 163.83 20.32 0)
+    (property "LCSC#" "C14663" (at 163.83 20.32 0)
       (effects (font (size 1.27 1.27)) hide)
     )
@@
       (effects (font (size 1.27 1.27)) hide)
     )
-    (property "JLC" "C14663" (at 172.72 20.32 0)
+    (property "LCSC#" "C14663" (at 172.72 20.32 0)
       (effects (font (size 1.27 1.27)) hide)
     )
@@
       (effects (font (size 1.27 1.27)) hide)
     )
-    (property "JLC" "C14663" (at 180.34 20.32 0)
+    (property "LCSC#" "C14663" (at 180.34 20.32 0)
       (effects (font (size 1.27 1.27)) hide)
     )
@@
       (effects (font (size 1.27 1.27)) hide)
     )
-    (property "JLC" "C14663" (at 189.23 20.32 0)
-      (effects (font (size 1.27 1.27)) hide)
-    )
+    (property "LCSC#" "C14663" (at 189.23 20.32 0)
+      (effects (font (size 1.27 1.27)) hide)
+    )
