File: Hardware/RP2040_Mini_PMod/RP2040_Mini_PMod.kicad_pcb (KiCad board)
At the start: 4 copper layers, 40 x 20 mm, 44 parts, among them J1 Micro_SD_Card, J3 Conn_02x06_Odd_Even, J4 USB_C_Receptacle_USB2.0, SW1 PTS815 SJK 250 SMTR LFS, SW2 PTS815 SJK 250 SMTR LFS, U1 RP2040, U2 W25Q128JVS, U3 NCP1117-3.3_SOT223, Y1 12MHz

Commit message: change reference for logo
Parts:
- renumbered G*** to G1
Changed lines of the file:
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@@
     (at 155.9 104.15 -90)
     (attr through_hole)
-    (fp_text reference "G***" (at 0 0 90) (layer "B.SilkS") hide
+    (fp_text reference "G1" (at 0 0 90) (layer "B.SilkS") hide
         (effects (font (size 1.524 1.524) (thickness 0.3)) (justify mirror))
     )

Commit message: change REF to Mount
Parts:
- renumbered REF** to Mount1
Changed lines of the file:
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@@
     (tags "mounting hole 2.2mm no annular m2")
     (attr exclude_from_pos_files exclude_from_bom)
-    (fp_text reference "REF**" (at 0 -3.2) (layer "F.SilkS") hide
+    (fp_text reference "Mount1" (at 0 -3.2) (layer "F.SilkS") hide
         (effects (font (size 1 1) (thickness 0.15)))
     )
@@
     (tags "mounting hole 2.2mm no annular m2")
     (attr exclude_from_pos_files exclude_from_bom)
-    (fp_text reference "REF**" (at -4.7 -1) (layer "F.SilkS") hide
-        (effects (font (size 1 1) (thickness 0.15)))
-    )
+    (fp_text reference "Mount1" (at -4.7 -1) (layer "F.SilkS") hide
+        (effects (font (size 1 1) (thickness 0.15)))
+    )
