File: Hardware/Pico_PMod/pico_pmod_host.kicad_pcb (KiCad board)
At the start: 2 copper layers, 66 x 43.2 mm, 10 parts, among them J1 Conn_02x15_Odd_Even, J2 Conn_01x02, J3 Conn_01x02, J4 Conn_01x02, J5 Conn_01x03, J7 Conn_01x05, SW1 SW_Push, U1 Pico

Commit message: update PCB to kicad7
Parts:
- renumbered G*** to Logo1
Other:
- net class Default removed
