File: Hardware/Pico_PMod/pico_pmod_host.kicad_pcb (KiCad board)
At the start: 2 copper layers, 66 x 43.2 mm, 10 parts, among them J1 Conn_02x15_Odd_Even, J2 Conn_01x02, J3 Conn_01x02, J4 Conn_01x02, J5 Conn_01x03, J7 Conn_01x05, SW1 SW_Push, U1 Pico

Commit message: update the logo reference
Parts:
- renumbered G*** to Logo2
Changed lines of the file:
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@@
     (at 147.3 85.7 180)
     (attr through_hole)
-    (fp_text reference "G***" (at 0 0) (layer "B.SilkS") hide
+    (fp_text reference "Logo2" (at 0 0) (layer "B.SilkS") hide
         (effects (font (size 1.524 1.524) (thickness 0.3)) (justify mirror))
     )
